File: assemble/assemble.kicad_pcb (KiCad board)
At the start: 2 copper layers, 262.4 x 104.6 mm, 125 parts, among them J1 Conn_01x04, J2 Conn_01x05, SW1 SW_Push, SW10 SW_Push, SW11 SW_Push, SW12 SW_Push, SW13 SW_Push, SW14 SW_Push, SW15 SW_Push, SW16 SW_Push, SW17 SW_Push, SW18 SW_Push, SW19 SW_Push, SW2 SW_Push, SW20 SW_Push, SW21 SW_Push, SW22 SW_Push, SW23 SW_Push, SW24 SW_Push, SW25 SW_Push, SW26 RotaryEncoder_Switch, SW27 SW_Push, SW28 SW_Push, SW29 SW_Push, SW3 SW_Push, SW30 SW_Push, SW31 SW_Push, SW32 SW_SPDT, SW33 SW_Push, SW34 SW_Push, SW35 SW_Push, SW36 SW_Push, SW37 SW_Push, SW38 SW_Push, SW39 RotaryEncoder_Switch, SW4 SW_Push, SW40 SW_Push, SW41 SW_Push, SW42 SW_Push, SW43 SW_Push, SW44 SW_Push, SW45 SW_Push, SW46 SW_Push, SW47 SW_Push, SW5 SW_Push, SW6 SW_Push, SW7 SW_Push, SW8 SW_Push, SW9 SW_Push, U1 XIAO-nRF52840-SMD, U2 XIAO-nRF52840-SMD

Commit message: feat: PCB renewal
Parts:
- removed Ref** (x6): Val**, kbd_Hole:m3_Screw_Hole_EdgeCuts
- J2: footprint Connector_PinHeader_2.00mm:PinHeader_1x05_P2.00mm_Vertical -> Connector_PinSocket_2.54mm:PinSocket_1x05_P2.54mm_Vertical
- JP1, JP2, U1, U2: moved to F.Cu
- R1, R2: footprint Resistor_SMD:R_0603_1608Metric_Pad0.98x0.95mm_HandSolder -> Resistor_THT:R_Axial_DIN0204_L3.6mm_D1.6mm_P5.08mm_Horizontal; moved to F.Cu
- SW26, SW39: value RotaryEncoder_Switch -> SW_Push; footprint kbd_Parts:RotaryEncoder_EC12E -> kicad-lib:Choc_v2_Hotswap_1u_16.6
- SW32: value SW_SPDT -> SW_Push; footprint kbd_Parts:TGSW_MSK-12D19 -> kicad-lib:Choc_v2_Hotswap_1u_16.6
- SW43: value SW_Push -> RotaryEncoder_Switch; footprint kicad-lib:Choc_v2_Hotswap_1u_16.6 -> kbd_Parts:RotaryEncoder_EC12E
- SW44: value SW_Push -> SW_SPDT; footprint kicad-lib:Choc_v2_Hotswap_1u_16.6 -> kbd_Parts:TGSW_MSK-12D19
- SW45: footprint kicad-lib:Choc_v2_Hotswap_1u_16.6 -> kbd_Parts:ResetSW
- SW46: value SW_Push -> RotaryEncoder_Switch; footprint kbd_Parts:ResetSW -> kbd_Parts:RotaryEncoder_EC12E
- moved SW46 176.1 mm to (235.8, 97.0), turned to 90 degrees
- moved D56 175.7 mm to (86.4, 90.4), turned to -90 degrees
- moved D57 162.0 mm to (102.0, 97.0), turned to -90 degrees
- moved SW32 160.8 mm to (119.8, 72.0), turned to -22.62 degrees
- moved SW37 154.9 mm to (91.7, 96.2), turned to -22.62 degrees
- moved D58 149.0 mm to (116.6, 103.0), turned to -90 degrees
- moved SW45 146.2 mm to (74.8, 176.0), turned to 0 degrees
- moved SW38 141.9 mm to (107.0, 102.6), turned to -22.62 degrees
- moved SW17 135.7 mm to (245.7, 40.9), turned to 0 degrees
- moved J2 132.6 mm to (244.4, 121.7), turned to 0 degrees
- moved SW44 132.5 mm to (279.9, 20.1), turned to 90 degrees
- moved D27 128.9 mm to (241.0, 37.2), turned to -90 degrees
- moved SW20 128.2 mm to (209.2, 42.6), turned to 22.62 degrees
- moved SW26 125.6 mm to (185.2, 88.6), turned to 22.62 degrees
- moved SW19 121.2 mm to (193.9, 49.0), turned to 22.62 degrees
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Connections:
- AE-XCL102D333CR-G1 pad 3: Net-(SW32-B) -> Net-(SW44-B)
- JP1 pad 1: RX_L -> TX_L
- JP1 pad 2: TX_R -> RX_R
- JP2 pad 1: TX_L -> RX_L
- JP2 pad 2: RX_R -> TX_R
- SW27 pad 1: Net-(D1-K) -> Net-(D13-K)
- SW27 pad 2: Net-(D37-A) -> Net-(D38-A)
- SW28 pad 1: Net-(D13-K) -> Net-(D19-K)
- SW28 pad 2: Net-(D38-A) -> Net-(D39-A)
- SW29 pad 1: Net-(D19-K) -> Net-(D25-K)
- SW29 pad 2: Net-(D39-A) -> Net-(D40-A)
- SW30 pad 1: Net-(D25-K) -> Net-(D31-K)
- SW30 pad 2: Net-(D40-A) -> Net-(D41-A)
- SW31 pad 1: Net-(D31-K) -> Net-(D44-K)
- SW31 pad 2: Net-(D41-A) -> Net-(D48-A)
- SW32 pad 1: unconnected-(SW32-A-Pad1) -> Net-(D45-K)
- SW32 pad 2: Net-(SW32-B) -> Net-(D49-A)
- SW33 pad 1: Net-(D44-K) -> Net-(D46-K)
- SW33 pad 2: Net-(D48-A) -> Net-(D50-A)
- SW34 pad 1: Net-(D45-K) -> Net-(D43-K)
- SW34 pad 2: Net-(D49-A) -> Net-(D52-A)
- SW35 pad 1: Net-(D46-K) -> Net-(D45-K)
- SW35 pad 2: Net-(D50-A) -> Net-(D53-A)
- SW36 pad 1: Net-(D43-K) -> Net-(D46-K)
- SW36 pad 2: Net-(D52-A) -> Net-(D54-A)
- SW37 pad 1: Net-(D45-K) -> Net-(D43-K)
- SW37 pad 2: Net-(D53-A) -> Net-(D56-A)
- SW38 pad 1: Net-(D46-K) -> Net-(D44-K)
- SW38 pad 2: Net-(D54-A) -> Net-(D57-A)
- SW40 pad 2: Net-(D56-A) -> Net-(D60-A)
- SW41 pad 2: Net-(D57-A) -> Net-(D61-A)
- SW42 pad 1: Net-(D46-K) -> Net-(D45-K)
- SW42 pad 2: Net-(D58-A) -> Net-(D62-A)
- SW44 pad 1: Net-(D44-K) -> unconnected-(SW44-A-Pad1)
- SW44 pad 2: Net-(D61-A) -> Net-(SW44-B)
- SW45 pad 1: Net-(D45-K) -> RST_GND_L
- SW45 pad 2: Net-(D62-A) -> RST_L
Routing:
- net BAT-: track 385.8 -> 0.00 mm, vias 8 -> 0
- net Net-(D31-K): track 359.4 -> 0.00 mm, vias 16 -> 0
- net PIN3L: track 357.0 -> 0.00 mm, vias 12 -> 0
- net BAT+: track 340.7 -> 0.00 mm, vias 6 -> 0
- net Net-(D42-K): track 303.3 -> 0.00 mm, vias 18 -> 0
- net PIN1L: track 298.5 -> 0.00 mm, vias 18 -> 0
- net Net-(D25-K): track 288.0 -> 0.00 mm, vias 14 -> 0
- net Net-(D19-K): track 285.9 -> 0.00 mm, vias 14 -> 0
- net Net-(D13-K): track 280.5 -> 0.00 mm, vias 12 -> 0
- net PIN2L: track 272.8 -> 0.00 mm, vias 14 -> 0
- net PIN6L: track 269.2 -> 0.00 mm, vias 11 -> 0
- net GNDR: track 261.8 -> 0.00 mm, vias 7 -> 0
- net Net-(D1-K): track 260.0 -> 0.00 mm, vias 18 -> 0
- net PIN1R: track 256.3 -> 0.00 mm, vias 12 -> 0
- net PIN5L: track 253.5 -> 0.00 mm, vias 14 -> 0
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Other:
- board outline removed
- board text removed: "ON"

Commit message: feat: implement version 2
Parts:
- added Ref**: Val**, kbd_Hole:m3_Screw_Hole_EdgeCuts, F.Cu at (101.0, 30.0)
- added Ref**: Val**, kbd_Hole:m3_Screw_Hole_EdgeCuts, F.Cu at (138.8, 113.4)
- added Ref**: Val**, kbd_Hole:m3_Screw_Hole_EdgeCuts, F.Cu at (162.8, 55.0)
- added Ref**: Val**, kbd_Hole:m3_Screw_Hole_EdgeCuts, F.Cu at (162.8, 113.8)
- added Ref**: Val**, kbd_Hole:m3_Screw_Hole_EdgeCuts, F.Cu at (200.6, 30.0)
- added Ref**: Val**, kbd_Hole:m3_Screw_Hole_EdgeCuts, F.Cu at (138.8, 55.0)
- JP1, JP2: moved to B.Cu
- R1, R2: footprint Resistor_THT:R_Axial_DIN0204_L3.6mm_D1.6mm_P5.08mm_Horizontal -> Resistor_SMD:R_0805_2012Metric_Pad1.20x1.40mm_HandSolder; moved to B.Cu
- moved J2 145.1 mm to (134.1, 27.4)
- moved J1 128.8 mm to (147.0, 55.6), turned to 90 degrees
- moved R1 124.6 mm to (154.8, 62.6), turned to 90 degrees
- moved R2 116.5 mm to (150.4, 62.6), turned to 90 degrees
- moved JP2 83.0 mm to (150.8, 106.8)
- moved JP1 72.9 mm to (150.8, 110.8)
- moved SW45 64.6 mm to (65.9, 112.0)
- moved SW47 63.1 mm to (235.8, 112.0)
- moved U2 41.6 mm to (269.7, 112.0)
- moved U1 39.4 mm to (32.0, 112.0)
- moved BT1 17.0 mm to (191.8, 32.8)
- moved D25 15.6 mm to (165.8, 71.4)
- moved D31 9.68 mm to (165.8, 79.6)
- moved D59 9.30 mm to (165.4, 97.4)
- moved SW44 8.64 mm to (282.4, 28.4), turned to -90 degrees
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Routing:
- net BAT-: track 0.00 -> 359.9 mm, vias 0 -> 3
- net Net-(D25-K): track 0.00 -> 333.3 mm, vias 0 -> 23
- net Net-(D31-K): track 0.00 -> 331.6 mm, vias 0 -> 14
- net BAT+: track 0.00 -> 328.1 mm, vias 0 -> 4
- net Net-(D43-K): track 0.00 -> 318.1 mm, vias 0 -> 19
- net Net-(D13-K): track 0.00 -> 314.5 mm, vias 0 -> 20
- net Net-(D19-K): track 0.00 -> 297.8 mm, vias 0 -> 18
- net PIN4L: track 0.00 -> 297.5 mm, vias 0 -> 13
- net Net-(D42-K): track 0.00 -> 297.4 mm, vias 0 -> 18
- net SDA: track 0.00 -> 293.9 mm, vias 0 -> 9
- net Net-(D44-K): track 0.00 -> 288.9 mm, vias 0 -> 13
- net Net-(D45-K): track 0.00 -> 288.2 mm, vias 0 -> 10
- net SCL: track 0.00 -> 280.7 mm, vias 0 -> 7
- net GNDR: track 0.00 -> 261.4 mm, vias 0 -> 8
- net Net-(D1-K): track 0.00 -> 261.1 mm, vias 0 -> 15
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Other:
- board outline added: 267 x 107 mm
- board text added: "Planetes42 v2"
