File: switch_plate/switch_plate.kicad_pcb (KiCad board)
At the start: 2 copper layers, 255 x 99.8 mm, 44 parts, among them SW1 SW_Push, SW10 SW_Push, SW11 SW_Push, SW12 SW_Push, SW13 SW_Push, SW14 SW_Push, SW15 SW_Push, SW16 SW_Push, SW17 SW_Push, SW18 SW_Push, SW19 SW_Push, SW2 SW_Push, SW20 SW_Push, SW21 SW_Push, SW22 SW_Push, SW23 SW_Push, SW24 SW_Push, SW25 SW_Push, SW27 SW_Push, SW28 SW_Push, SW29 SW_Push, SW3 SW_Push, SW30 SW_Push, SW31 SW_Push, SW33 SW_Push, SW34 SW_Push, SW35 SW_Push, SW36 SW_Push, SW37 SW_Push, SW38 SW_Push, SW4 SW_Push, SW40 SW_Push, SW41 SW_Push, SW42 SW_Push, SW43 SW_Push, SW44 SW_Push, SW45 SW_Push, SW5 SW_Push, SW6 SW_Push, SW7 SW_Push, SW8 SW_Push, SW9 SW_Push

Commit message: refactor: start re-wiring
Other:
- outline, holes or cut-outs redrawn
Changed lines of the file:
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@@
 	)
 	(gr_line
-		(start 134.8 54.6)
-		(end 134.8 72.4)
+		(start 134.8 72.4)
+		(end 134.8 57)
 		(stroke
 			(width 0.05)
@@
 	(gr_line
 		(start 86.4 44.6)
-		(end 125.6 54.6)
+		(end 134.8 57)
 		(stroke
 			(width 0.05)
@@
 	)
 	(gr_line
-		(start 160.4 72.4)
-		(end 160.4 54.6)
+		(start 161.4 72.4)
+		(end 161.4 57)
 		(stroke
 			(width 0.05)
@@
 		(start 21.6 38.8)
 		(end 86.4 38.8)
-		(stroke
-			(width 0.05)
-			(type default)
-		)
-		(layer "Edge.Cuts")
-	)
-	(gr_line
-		(start 125.6 54.6)
-		(end 134.8 54.6)
 		(stroke
 			(width 0.05)
@@
 	)
 	(gr_line
-		(start 160.4 54.6)
+		(start 161.4 57)
 		(end 209.2 45.2)
 		(stroke
@@
 	(gr_line
 		(start 134.8 72.4)
-		(end 160.4 72.4)
+		(end 161.4 72.4)
 		(stroke
 			(width 0.05)

Commit message: fix: update switch plate
Parts:
- moved SW8 1.80 mm to (67.7, 74.6)
- moved SW3 1.80 mm to (31.2, 91.2)
- moved SW1 1.80 mm to (37.8, 58.0)
- moved SW10 1.80 mm to (90.9, 58.0)
- moved SW11 1.80 mm to (87.6, 74.6)
- moved SW12 1.80 mm to (84.3, 91.2)
- moved SW13 1.80 mm to (106.2, 64.4)
- moved SW14 1.80 mm to (102.9, 81.0)
- moved SW15 1.80 mm to (99.6, 97.6)
- moved SW16 1.80 mm to (121.6, 70.8)
- moved SW17 1.80 mm to (118.2, 87.4)
- moved SW18 1.80 mm to (114.9, 104.0)
- moved SW19 1.80 mm to (90.2, 111.6)
- moved SW2 1.80 mm to (34.5, 74.6)
- moved SW20 1.80 mm to (105.5, 118.0)
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Other:
- outline, holes or cut-outs redrawn
Changed lines of the file:
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@@
 		(tenting front back)
 		(pcbplotparams
-			(layerselection 0x00000000_00000000_55555555_5755f5ff)
+			(layerselection 0x00000000_00000000_55555555_575555f0)
 			(plot_on_all_layers_selection 0x00000000_00000000_00000000_00000000)
 			(disableapertmacros no)
@@
 			(drillshape 0)
 			(scaleselection 1)
-			(outputdirectory "../jclpcb/")
+			(outputdirectory "../jclpcb_20250728/")
 		)
 	)
@@
 	(footprint "kicad-lib:SW_Hole_1u_16.6"
 		(layer "F.Cu")
-		(at 32.68 74.6 180)
+		(at 34.48 74.6 180)
 		(property "Reference" "SW2"
 			(at -0.15 -0.5 180)
@@
 	(footprint "kicad-lib:SW_Hole_1u_16.6"
 		(layer "F.Cu")
-		(at 118.999922 124.400035 -22.62)
+		(at 120.799922 124.400035 -22.62)
 		(property "Reference" "SW21"
 			(at -0.15 -0.5 337.38)
@@
 	(footprint "kicad-lib:SW_Hole_1u_16.6"
 		(layer "F.Cu")
-		(at 104.44314 64.384616 -22.62)
+		(at 106.24314 64.384616 -22.62)
 		(property "Reference" "SW13"
 			(at -0.15 -0.5 337.38)
@@
 	(footprint "kicad-lib:SW_Hole_1u_16.6"
 		(layer "F.Cu")
-		(at 65.88 74.6)
+		(at 67.68 74.6)
 		(property "Reference" "SW8"
 			(at -0.15 -0.5 0)
@@
 	(footprint "kicad-lib:SW_Hole_1u_16.6"
 		(layer "F.Cu")
-		(at 69.2 58)
+		(at 71 58)
 		(property "Reference" "SW7"
 			(at -0.15 -0.5 0)
@@
 	(footprint "kicad-lib:SW_Hole_1u_16.6"
 		(layer "F.Cu")
-		(at 88.353798 111.630732 -22.62)
+		(at 90.153798 111.630732 -22.62)
 		(property "Reference" "SW19"
 			(at -0.15 -0.5 337.38)
@@
 	(footprint "kicad-lib:SW_Hole_1u_16.6"
 		(layer "F.Cu")
-		(at 36 58 180)
+		(at 37.8 58 180)
 		(property "Reference" "SW1"
 			(at -0.15 -0.5 180)
@@
 	(footprint "kicad-lib:SW_Hole_1u_16.6"
 		(layer "F.Cu")
-		(at 82.48 91.199949 -22.62)
+		(at 84.28 91.199949 -22.62)
 		(property "Reference" "SW12"
 			(at -0.15 -0.5 337.38)
@@
 	(footprint "kicad-lib:SW_Hole_1u_16.6"
 		(layer "F.Cu")
-		(at 62.56 91.2)
+		(at 64.36 91.2)
 		(property "Reference" "SW9"
 			(at -0.15 -0.5 0)
@@
 	(footprint "kicad-lib:SW_Hole_1u_16.6"
 		(layer "F.Cu")
-		(at 119.766202 70.769268 -22.62)
+		(at 121.566202 70.769268 -22.62)
 		(property "Reference" "SW16"
 			(at -0.15 -0.5 337.38)
@@
 	(footprint "kicad-lib:SW_Hole_1u_16.6"
 		(layer "F.Cu")
-		(at 52.6 58)
+		(at 54.4 58)
 		(property "Reference" "SW4"
 			(at -0.15 -0.5 0)
@@
 	(footprint "kicad-lib:SW_Hole_1u_16.6"
 		(layer "F.Cu")
-		(at 116.446163 87.36926 -22.62)
+		(at 118.246163 87.36926 -22.62)
 		(property "Reference" "SW17"
 			(at -0.15 -0.5 337.38)
@@
 	(footprint "kicad-lib:SW_Hole_1u_16.6"
 		(layer "F.Cu")
-		(at 101.123101 80.984608 -22.62)
+		(at 102.923101 80.984608 -22.62)
 		(property "Reference" "SW14"
 			(at -0.15 -0.5 337.38)
@@
 	(footprint "kicad-lib:SW_Hole_1u_16.6"
 		(layer "F.Cu")
-		(at 85.800039 74.599957 -22.62)
+		(at 87.600039 74.599957 -22.62)
 		(property "Reference" "SW11"
 			(at -0.15 -0.5 337.38)
@@
 	(footprint "kicad-lib:SW_Hole_1u_16.6"
 		(layer "F.Cu")
-		(at 97.803062 97.584601 -22.62)
+		(at 99.603062 97.584601 -22.62)
 		(property "Reference" "SW15"
 			(at -0.15 -0.5 337.38)
@@
 	(footprint "kicad-lib:SW_Hole_1u_16.6"
 		(layer "F.Cu")
-		(at 103.67686 118.015384 -22.62)
+		(at 105.47686 118.015384 -22.62)
 		(property "Reference" "SW20"
 			(at -0.15 -0.5 337.38)
@@
 	(footprint "kicad-lib:SW_Hole_1u_16.6"
 		(layer "F.Cu")
-		(at 113.126124 103.969252 -22.62)
+		(at 114.926124 103.969252 -22.62)
 		(property "Reference" "SW18"
 			(at -0.15 -0.5 337.38)
@@
 	(footprint "kicad-lib:SW_Hole_1u_16.6"
 		(layer "F.Cu")
-		(at 89.120078 57.999965 -22.62)
+		(at 90.920078 57.999965 -22.62)
 		(property "Reference" "SW10"
 			(at -0.15 -0.5 337.38)
@@
 	(footprint "kicad-lib:SW_Hole_1u_16.6"
 		(layer "F.Cu")
-		(at 49.28 74.6)
+		(at 51.08 74.6)
 		(property "Reference" "SW5"
 			(at -0.15 -0.5 0)
@@
 	(footprint "kicad-lib:SW_Hole_1u_16.6"
 		(layer "F.Cu")
-		(at 45.96 91.2)
+		(at 47.76 91.2)
 		(property "Reference" "SW6"
 			(at -0.15 -0.5 0)
@@
 	(footprint "kicad-lib:SW_Hole_1u_16.6"
 		(layer "F.Cu")
-		(at 29.36 91.2 180)
+		(at 31.16 91.2 180)
 		(property "Reference" "SW3"
 			(at -0.15 -0.5 180)
@@
 	)
 	(gr_line
-		(start 86.4 38.8)
-		(end 86.4 44.6)
+		(start 87.6 46.8)
+		(end 133 65.8)
 		(stroke
 			(width 0.05)
@@
 	)
 	(gr_line
-		(start 134.8 72.4)
-		(end 134.8 57)
+		(start 226.3 105.3)
+		(end 241.4 105.3)
 		(stroke
 			(width 0.05)
@@
 	)
 	(gr_line
-		(start 20.6 39.8)
+		(start 208.6 42.2)
+		(end 208.6 38.8)
+		(stroke
+			(width 0.05)
+			(type default)
+		)
+		(layer "Edge.Cuts")
+	)
+	(gr_line
+		(start 133 65.8)
+		(end 133 73.8)
+		(stroke
+			(width 0.05)
+			(type default)
+		)
+		(layer "Edge.Cuts")
+	)
+	(gr_line
+		(start 20.6 72.8)
 		(end 20.6 137.6)
 		(stroke
@@
 	)
 	(gr_line
-		(start 86.4 44.6)
-		(end 134.8 57)
+		(start 70 105.3)
+		(end 70 123.9)
 		(stroke
 			(width 0.05)
@@
 	)
 	(gr_line
-		(start 21.6 138.6)
-		(end 274.6 138.6)
+		(start 87.6 38.8)
+		(end 47.6 38.8)
 		(stroke
 			(width 0.05)
@@
 		(layer "Edge.Cuts")
 	)
-	(gr_rect
-		(start 55.6 125)
-		(end 65.6 129.6)
+	(gr_line
+		(start 54.7 105.3)
+		(end 70 105.3)
+		(stroke
+			(width 0.05)
+			(type default)
+		)
+		(layer "Edge.Cuts")
+	)
+	(gr_line
+		(start 241.4 123.9)
+		(end 226.3 123.9)
 		(stroke
 			(width 0.05)
 			(type default)
 		)
-		(fill no)
 		(layer "Edge.Cuts")
 	)
 	(gr_line
-		(start 161.4 72.4)
-		(end 161.4 57)
+		(start 47.6 38.8)
+		(end 21.6 38.8)
 		(stroke
 			(width 0.05)
@@
 	)
 	(gr_line
-		(start 21.6 38.8)
-		(end 86.4 38.8)
+		(start 87.6 42.2)
+		(end 87.6 46.8)
 		(stroke
 			(width 0.05)
@@
 	(gr_rect
 		(start 228.6 125)
-		(end 239.2 129.8)
+		(end 239 129.8)
 		(stroke
 			(width 0.05)
@@
 	)
 	(gr_line
-		(start 209.2 38.8)
-		(end 274.6 38.8)
+		(start 163 66)
+		(end 208.6 46.6)
 		(stroke
 			(width 0.05)
@@
 	)
 	(gr_line
-		(start 209.2 38.8)
-		(end 209.2 45.2)
+		(start 21.6 138.6)
+		(end 274.6 138.6)
+		(stroke
+			(width 0.05)
+			(type default)
+		)
+		(layer "Edge.Cuts")
+	)
+	(gr_line
+		(start 208.6 38.8)
+		(end 274.6 38.8)
 		(stroke
 			(width 0.05)
@@
 		(layer "Edge.Cuts")
 	)
+	(gr_line
+		(start 226.3 105.3)
+		(end 226.3 123.9)
+		(stroke
+			(width 0.05)
+			(type default)
+		)
+		(layer "Edge.Cuts")
+	)
+	(gr_line
+		(start 163 73.8)
+		(end 163 66)
+		(stroke
+			(width 0.05)
+			(type default)
+		)
+		(layer "Edge.Cuts")
+	)
+	(gr_line
+		(start 208.6 42.2)
+		(end 208.6 46.6)
+		(stroke
+			(width 0.05)
+			(type default)
+		)
+		(layer "Edge.Cuts")
+	)
 	(gr_arc
 		(start 274.6 38.8)
@@
 	)
 	(gr_line
-		(start 275.6 137.6)
-		(end 275.6 39.8)
+		(start 20.6 72.8)
+		(end 20.6 39.8)
 		(stroke
 			(width 0.05)
@@
 		(layer "Edge.Cuts")
 	)
-	(gr_rect
-		(start 226 105.2)
-		(end 242 123.8)
+	(gr_line
+		(start 241.4 105.3)
+		(end 241.4 123.9)
+		(stroke
+			(width 0.05)
+			(type default)
+		)
+		(layer "Edge.Cuts")
+	)
+	(gr_line
+		(start 70 123.9)
+		(end 54.7 123.9)
 		(stroke
 			(width 0.05)
 			(type default)
 		)
-		(fill no)
 		(layer "Edge.Cuts")
 	)
@@
 		(layer "Edge.Cuts")
 	)
+	(gr_rect
+		(start 57.6 125.2)
+		(end 67 129.4)
+		(stroke
+			(width 0.05)
+			(type default)
+		)
+		(fill no)
+		(layer "Edge.Cuts")
+	)
+	(gr_line
+		(start 54.7 105.3)
+		(end 54.7 123.9)
+		(stroke
+			(width 0.05)
+			(type default)
+		)
+		(layer "Edge.Cuts")
+	)
 	(gr_arc
 		(start 21.6 138.6)
@@
 	)
 	(gr_line
-		(start 161.4 57)
-		(end 209.2 45.2)
+		(start 133 73.8)
+		(end 163 73.8)
 		(stroke
 			(width 0.05)
@@
 	)
 	(gr_line
-		(start 134.8 72.4)
-		(end 161.4 72.4)
+		(start 275.6 137.6)
+		(end 275.6 39.8)
 		(stroke
 			(width 0.05)
@@
 		(layer "Edge.Cuts")
 	)
-	(gr_rect
-		(start 53 105.2)
-		(end 68 124)
+	(gr_line
+		(start 87.6 42.2)
+		(end 87.6 38.8)
 		(stroke
 			(width 0.05)
 			(type default)
 		)
-		(fill no)
 		(layer "Edge.Cuts")
 	)

Commit message: feat: update switch plate
Parts:
- removed the Ref** at (154.0, 130.0)
- removed the Ref** at (141.2, 130.0)
- removed SW43, SW44, SW45: SW_Push, kicad-lib:SW_Hole_1u_16.6
- added Ref**: Val**, kbd_Hole:m3_Spacer_Hole, F.Cu at (138.8, 113.4)
- added Ref**: Val**, kbd_Hole:m3_Spacer_Hole, F.Cu at (162.8, 113.8)
- added SW26: SW_Push, kicad-lib:SW_Hole_1u_16.6, F.Cu at (185.2, 88.6)
- added SW32: SW_Push, kicad-lib:SW_Hole_1u_16.6, F.Cu at (119.8, 72.0)
- added SW39: SW_Push, kicad-lib:SW_Hole_1u_16.6, F.Cu at (122.4, 109.0)
- moved SW37 154.9 mm to (91.7, 96.2), turned to -22.62 degrees
- moved SW38 141.9 mm to (107.0, 102.6), turned to -22.62 degrees
- moved SW17 135.7 mm to (245.7, 40.9), turned to 0 degrees
- moved SW20 128.2 mm to (209.2, 42.6), turned to 22.62 degrees
- moved SW19 121.2 mm to (193.9, 49.0), turned to 22.62 degrees
- moved SW33 112.9 mm to (116.5, 88.6), turned to -22.62 degrees
- moved SW16 111.6 mm to (229.1, 40.9), turned to 0 degrees
- moved SW31 95.8 mm to (123.1, 55.4), turned to -22.62 degrees
- moved SW40 94.1 mm to (179.3, 109.0), turned to 22.62 degrees
- moved SW21 80.5 mm to (181.9, 72.0), turned to 22.62 degrees
- moved SW18 80.1 mm to (178.6, 55.4), turned to 22.62 degrees
- moved SW41 72.7 mm to (194.6, 102.6), turned to 22.62 degrees
- moved SW24 69.1 mm to (232.4, 57.5), turned to 0 degrees
- moved SW3 65.1 mm to (72.6, 40.9)
- moved SW5 62.2 mm to (107.8, 49.0), turned to 157.38 degrees
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Other:
- board size 255 x 99.8 mm -> 258.8 x 101 mm
