File: assemble_v3/assemble_v3.kicad_pcb (KiCad board)
At the start: 2 copper layers, 267 x 107 mm, 121 parts, among them J1 Conn_01x04, J2 Conn_01x05, SW1 SW_Push, SW10 SW_Push, SW11 SW_Push, SW12 SW_Push, SW13 SW_Push, SW14 SW_Push, SW15 SW_Push, SW16 SW_Push, SW17 SW_Push, SW18 SW_Push, SW19 SW_Push, SW2 SW_Push, SW20 SW_Push, SW21 SW_Push, SW22 SW_Push, SW23 SW_Push, SW24 SW_Push, SW25 SW_Push, SW26 SW_Push, SW27 SW_Push, SW28 SW_Push, SW29 SW_Push, SW3 SW_Push, SW30 SW_Push, SW31 SW_Push, SW32 SW_Push, SW33 SW_Push, SW34 SW_Push, SW35 SW_Push, SW36 SW_Push, SW37 SW_Push, SW38 SW_Push, SW39 SW_Push, SW4 SW_Push, SW40 SW_Push, SW41 SW_Push, SW42 SW_Push, SW43 RotaryEncoder_Switch, SW44 SW_SPDT, SW45 RotaryEncoder_Switch, SW5 SW_Push, SW6 SW_Push, SW7 SW_Push, SW8 SW_Push, SW9 SW_Push, U1 XIAO-nRF52840-SMD, U2 XIAO-nRF52840-SMD

Commit message: feat: implement v3
Parts:
- J2: footprint Connector_PinHeader_2.54mm:PinHeader_1x05_P2.54mm_Vertical -> Connector_PinSocket_2.54mm:PinSocket_1x05_P2.54mm_Vertical
- moved D15 1.40 mm to (68.4, 51.6)
- moved D44 0.60 mm to (194.4, 78.6)
- moved D62 0.60 mm to (173.4, 105.0)
- moved D60 0.57 mm to (203.6, 92.6)
- moved D61 0.57 mm to (188.2, 99.0)
- moved D1 0.10 mm to (29.0, 88.4)
Routing:
- net BAT-: track 0.00 -> 363.4 mm, vias 0 -> 7
- net BAT+: track 0.00 -> 333.8 mm, vias 0 -> 6
- net GNDR: track 0.00 -> 292.0 mm, vias 0 -> 7
- net GNDL: track 0.00 -> 277.9 mm, vias 0 -> 6
- net VCCL: track 0.00 -> 245.2 mm, vias 0 -> 4
- net MOSI: track 0.00 -> 245.0 mm, vias 0 -> 3
- net VCCR: track 0.00 -> 236.6 mm, vias 0 -> 3
- net SCK: track 0.00 -> 226.8 mm, vias 0 -> 6
- net Net-(D35-K): track 0.00 -> 226.1 mm, vias 0 -> 12
- net Net-(D32-K): track 0.00 -> 224.6 mm, vias 0 -> 15
- net Net-(D11-K): track 0.00 -> 217.9 mm, vias 0 -> 14
- net Net-(D1-K): track 0.00 -> 203.5 mm, vias 0 -> 16
- net CS: track 0.00 -> 202.4 mm, vias 0 -> 3
- net PIN1R: track 0.00 -> 198.1 mm, vias 0 -> 14
- net Net-(D33-K): track 0.00 -> 190.5 mm, vias 0 -> 16
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Other:
- board text added: "Planetes42 v3"
